File: T08_rc360detector.brd (EAGLE design)
At the start: 100 x 80 mm, 55 parts, among them IC1 LM317MSTT3, IC2 LM317MSTT3, IC3 LM1117, U2 ATMEGA328P_PDIP, X1 SSW-101-02-S-D, X3 SSW-101-02-S-D, X4 87758-0616, X5 87758-0616, X6 SSW-104-02-S-Q

Commit message: Slight changes. Passed DRC
Made sure DRC worked and had updated libraries. This should work now,
(hopefully)
Connections:
- removed net TP8: SV1.9
- removed net TP9: SV1.10
- net GND: now also CX-0905C.OUT; no longer CX-0905C.P$2
- net N$4: now also CX-0905C.IN; no longer CX-0905C.P$1
Routing:
- net TWI_SCL: track 13.6 -> 14.1 mm, vias 1 -> 0
