File: T08_rc360detector.sch (EAGLE design)
At the start: 55 parts, among them IC1 LM317MSTT3, IC2 LM317MSTT3, IC3 LM1117, U2 ATMEGA328P_PDIP, X1 SSW-101-02-S-D, X3 SSW-101-02-S-D, X4 87758-0616, X5 87758-0616, X6 SSW-104-02-S-Q

Commit message: Slight changes. Passed DRC
Made sure DRC worked and had updated libraries. This should work now,
(hopefully)
Connections:
- removed net TP8: SV1.9
- removed net TP9: SV1.10
Changed lines of the file:
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@@
-</segment>
-</net>
-<net name="TP8" class="0">
-<segment>
-<pinref part="SV1" gate="G$1" pin="9"/>
-<wire x1="256.54" y1="190.5" x2="264.16" y2="190.5" width="0.1524" layer="91"/>
-<label x="259.08" y="190.5" size="1.778" layer="95"/>
-</segment>
-</net>
-<net name="TP9" class="0">
-<segment>
-<pinref part="SV1" gate="G$1" pin="10"/>
-<wire x1="256.54" y1="193.04" x2="264.16" y2="193.04" width="0.1524" layer="91"/>
-<label x="259.08" y="193.04" size="1.778" layer="95"/>
 </segment>
 </net>
